File: wegstr-wasteboard.kicad_pcb (KiCad board)
At the start: 2 copper layers, 198.3 x 138.4 mm, 0 parts

Commit message: Add "FRONT" text.
Other:
- board text added: "FRONT"
Changed lines of the file:
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@@
   (general
     (thickness 1.6)
-    (drawings 26)
+    (drawings 27)
     (tracks 0)
     (zones 0)
@@
     (uvia_drill 0.1)
   )
+  (gr_text FRONT (at 262.89 85.09 90) (layer Dwgs.User)
+    (effects (font (size 4 5) (thickness 0.5)))
+  )
   (gr_line (start 255.27 154.305) (end 56.938333 154.305) (layer Edge.Cuts) (width 0.15))
